File: ikoka-pro-meshtastic-device.kicad_pcb (KiCad board)
At the start: 2 copper layers, 80 x 100 mm, 63 parts, among them J1 Barrel_Jack_Switch, J10 BWSMA-KWE-Z001, J2 Conn_ARM_JTAG_SWD_10, J3 BWSMA-KWE-Z001, J4 Conn_01x01, J5 Conn_01x01, J6 Conn_01x01, J7 Conn_01x01, J8 USB_C_Receptacle_USB2.0_16P, SW2 TS36CA-0.6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

Commit message: feat: Move SWD pads further away from USB-C and battery
Signed-off-by: Andrew Yong <me@ndoo.sg>
Parts:
- moved J2 2.50 mm to (150.0, 122.5)
Routing:
- net ~{RESET}: track 49.9 -> 51.3 mm
- net SWDIO: track 32.7 -> 33.7 mm
- net SWCLK: track 35.6 -> 36.7 mm
- net GND: vias 168 -> 169
